File: CAN-RGB-1.kicad_pcb (KiCad board)
At the start: 2 copper layers, 26 parts, among them J1 Conn_01x06_Socket, J2 Conn_01x03_Socket, P1 USB_C_Plug_USB2.0, SW1 SW_Push, U2 ATmega32U4-A, U3 MCP2561-E_SN, Y1 16 MHz

Commit message: Layout connections mostly complete
Parts:
- moved R4 7.71 mm to (114.3, 61.0)
- moved SW1 6.11 mm to (121.9, 61.0)
- moved C2 2.78 mm to (109.6, 81.3)
- moved C7 2.60 mm to (154.6, 66.0)
- moved C3 2.46 mm to (118.0, 66.0)
- moved R5 2.46 mm to (113.5, 66.0)
- moved R1 2.34 mm to (110.0, 73.7)
- moved R6 2.26 mm to (153.7, 78.7)
- moved J1 1.80 mm to (159.5, 72.5)
- moved J2 1.62 mm to (159.5, 84.9)
- moved R2 1.30 mm to (110.0, 76.2)
- moved C5 1.24 mm to (151.3, 78.7)
- moved R7 1.22 mm to (153.7, 81.3)
- moved U2 0.80 mm to (118.5, 76.2)
- moved C1 0.76 mm to (110.2, 78.7)
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Routing:
- net GND: track 0.00 -> 88.6 mm, vias 0 -> 4
- net +5V: track 0.00 -> 55.1 mm, vias 0 -> 2
- net Net-(J2-Pin_1): track 0.00 -> 39.5 mm, vias 0 -> 2
- net DIO: track 0.00 -> 37.8 mm, vias 0 -> 1
- net CANL: track 0.00 -> 37.5 mm
- net +12V: track 0.00 -> 31.6 mm, vias 0 -> 4
- net RX: track 0.00 -> 29.5 mm, vias 0 -> 2
- net RST: track 0.00 -> 28.9 mm
- net TX: track 0.00 -> 28.7 mm, vias 0 -> 2
- net CANH: track 0.00 -> 22.9 mm, vias 0 -> 1
- net Net-(U2-XTAL2): track 0.00 -> 19.0 mm
- net Net-(U2-XTAL1): track 0.00 -> 16.6 mm, vias 0 -> 2
- net Net-(R5-Pad1): track 0.00 -> 15.6 mm, vias 0 -> 2
- net UGND: track 0.00 -> 12.9 mm, vias 0 -> 2
- net Net-(U2-VBUS): track 0.00 -> 9.00 mm
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