File: hardware/kicad/CANLED328p.kicad_pcb (KiCad board)
At the start: 2 copper layers, 83.5 x 59 mm, 35 parts, among them J1 2604-1103, J2 2604-1103, J3 AVR-ISP-6, J4 Conn_01x04_Socket, J5 Conn_01x02_Socket, J6 2604-1103, U1 MCP2515-I_SO, U2 TSR_1-2450, U3 MCP2561-E_SN, U4 ATmega328-P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

Commit message: Library added, files updated to use library
Parts:
- C1, C2, C5, C6, C7: footprint footprints:K104K10X7RF5UH5_VIS -> LibraryCANLED:K104K10X7RF5UH5_VIS
- C10: footprint Capacitor_THT:CP_Radial_D10.0mm_P5.00mm -> LibraryCANLED:CP_Radial_D10.0mm_P5.00mm
- C12, C13, C4, C8: footprint Capacitor_THT:C_Disc_D5.0mm_W2.5mm_P5.00mm -> LibraryCANLED:C_Disc_D5.0mm_W2.5mm_P5.00mm
- C3: footprint Capacitor_THT:C_Disc_D6.0mm_W2.5mm_P5.00mm -> LibraryCANLED:C_Disc_D6.0mm_W2.5mm_P5.00mm
- C9: footprint Capacitor_THT:CP_Radial_D5.0mm_P2.50mm -> LibraryCANLED:CP_Radial_D5.0mm_P2.50mm
- D1, D2: footprint LED_THT:LED_D4.0mm -> LibraryCANLED:LED_D4.0mm
- D3: footprint Diode_THT:D_DO-41_SOD81_P10.16mm_Horizontal -> LibraryCANLED:D_DO-41_SOD81_P10.16mm_Horizontal
- J1, J2, J6: footprint 2604-1103-1:CONN3_2604-1103_WAG -> LibraryCANLED:CONN3_2604-1103_WAG
- J3: footprint Connector_IDC:IDC-Header_2x03_P2.54mm_Vertical -> LibraryCANLED:IDC-Header_2x03_P2.54mm_Vertical
- J4: footprint 2604-1104-1:CONN4_2604-1104_WAG -> LibraryCANLED:CONN4_2604-1104_WAG
- J5: footprint Connector_PinHeader_2.54mm:PinHeader_1x02_P2.54mm_Vertical -> LibraryCANLED:PinHeader_1x02_P2.54mm_Vertical
- JP1: footprint Jumper:SolderJumper-2_P1.3mm_Open_Pad1.0x1.5mm -> LibraryCANLED:SolderJumper-2_P1.3mm_Open_Pad1.0x1.5mm
- L1: footprint Inductor_THT:L_Axial_L6.6mm_D2.7mm_P10.16mm_Horizontal_Vishay_IM-2 -> LibraryCANLED:L_Axial_L6.6mm_D2.7mm_P10.16mm_Horizontal_Vishay_IM-2
- R1, R2, R3, R4, R5: footprint Resistor_THT:R_Axial_DIN0207_L6.3mm_D2.5mm_P10.16mm_Horizontal -> LibraryCANLED:R_Axial_DIN0207_L6.3mm_D2.5mm_P10.16mm_Horizontal
- S1: footprint TS02_66_55_BK_100_LCR_D:SW_TS02-66-55-BK-100-LCR-D -> LibraryCANLED:SW_TS02-66-55-BK-100-LCR-D
- U1: footprint Package_DIP:DIP-18_W7.62mm_LongPads -> LibraryCANLED:DIP-18_W7.62mm_LongPads
- U2: footprint Converter_DCDC:Converter_DCDC_TRACO_TSR-1_THT -> LibraryCANLED:Converter_DCDC_TRACO_TSR-1_THT
- U3: footprint Package_DIP:DIP-8_W7.62mm_Socket_LongPads -> LibraryCANLED:DIP-8_W7.62mm_Socket_LongPads
- U4: footprint Package_DIP:DIP-28_W7.62mm -> LibraryCANLED:DIP-28_W7.62mm
- Y1, Y2: footprint ABL-16.000MHZ-B2:XTAL_HC49P488W46L1150T500H350 -> LibraryCANLED:XTAL_HC49P488W46L1150T500H350
Changed lines of the file:
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@@
 	(net 47 "SCL")
 	(net 48 "SDA")
-	(footprint "Resistor_THT:R_Axial_DIN0207_L6.3mm_D2.5mm_P10.16mm_Horizontal"
+	(footprint "LibraryCANLED:R_Axial_DIN0207_L6.3mm_D2.5mm_P10.16mm_Horizontal"
 		(layer "F.Cu")
 		(at 150.34 93)
@@
 		)
 	)
-	(footprint "Converter_DCDC:Converter_DCDC_TRACO_TSR-1_THT"
+	(footprint "LibraryCANLED:Converter_DCDC_TRACO_TSR-1_THT"
 		(layer "F.Cu")
 		(at 184 68.5)
@@
 		)
 	)
-	(footprint "Inductor_THT:L_Axial_L6.6mm_D2.7mm_P10.16mm_Horizontal_Vishay_IM-2"
+	(footprint "LibraryCANLED:L_Axial_L6.6mm_D2.7mm_P10.16mm_Horizontal_Vishay_IM-2"
 		(layer "F.Cu")
 		(at 158.92 71)
@@
 		)
 	)
-	(footprint "Package_DIP:DIP-8_W7.62mm_Socket_LongPads"
+	(footprint "LibraryCANLED:DIP-8_W7.62mm_Socket_LongPads"
 		(layer "F.Cu")
 		(at 136.38 64.38)
@@
 		)
 	)
-	(footprint "footprints:K104K10X7RF5UH5_VIS"
+	(footprint "LibraryCANLED:K104K10X7RF5UH5_VIS"
 		(layer "F.Cu")
 		(at 131.5 98.5 90)
@@
 		(embedded_fonts no)
 	)
-	(footprint "Capacitor_THT:CP_Radial_D5.0mm_P2.50mm"
+	(footprint "LibraryCANLED:CP_Radial_D5.0mm_P2.50mm"
 		(layer "F.Cu")
 		(at 126 77.5 90)
@@
 		)
 	)
-	(footprint "Resistor_THT:R_Axial_DIN0207_L6.3mm_D2.5mm_P10.16mm_Horizontal"
+	(footprint "LibraryCANLED:R_Axial_DIN0207_L6.3mm_D2.5mm_P10.16mm_Horizontal"
 		(layer "F.Cu")
 		(at 161.42 87.5)
@@
 		)
 	)
-	(footprint "footprints:K104K10X7RF5UH5_VIS"
+	(footprint "LibraryCANLED:K104K10X7RF5UH5_VIS"
 		(layer "F.Cu")
 		(at 186.5 84.5 180)
@@
 		(embedded_fonts no)
 	)
-	(footprint "footprints:K104K10X7RF5UH5_VIS"
+	(footprint "LibraryCANLED:K104K10X7RF5UH5_VIS"
 		(layer "F.Cu")
 		(at 182 75)
@@
 		(embedded_fonts no)
 	)
-	(footprint "ABL-16.000MHZ-B2:XTAL_HC49P488W46L1150T500H350"
+	(footprint "LibraryCANLED:XTAL_HC49P488W46L1150T500H350"
 		(layer "F.Cu")
 		(at 148.5 81.5 -90)
@@
 		(embedded_fonts no)
 	)
-	(footprint "TS02_66_55_BK_100_LCR_D:SW_TS02-66-55-BK-100-LCR-D"
+	(footprint "LibraryCANLED:SW_TS02-66-55-BK-100-LCR-D"
 		(layer "F.Cu")
 		(at 168 94.5)
@@
 		(embedded_fonts no)
 	)
-	(footprint "Resistor_THT:R_Axial_DIN0207_L6.3mm_D2.5mm_P10.16mm_Horizontal"
+	(footprint "LibraryCANLED:R_Axial_DIN0207_L6.3mm_D2.5mm_P10.16mm_Horizontal"
 		(layer "F.Cu")
 		(at 161.42 83.5)
@@
 		)
 	)
-	(footprint "Capacitor_THT:CP_Radial_D10.0mm_P5.00mm"
+	(footprint "LibraryCANLED:CP_Radial_D10.0mm_P5.00mm"
 		(layer "F.Cu")
 		(at 149.6323 68.5)
@@
 		)
 	)
-	(footprint "Resistor_THT:R_Axial_DIN0207_L6.3mm_D2.5mm_P10.16mm_Horizontal"
+	(footprint "LibraryCANLED:R_Axial_DIN0207_L6.3mm_D2.5mm_P10.16mm_Horizontal"
 		(layer "F.Cu")
 		(at 163.42 64.5)
@@
 		)
 	)
-	(footprint "footprints:K104K10X7RF5UH5_VIS"
+	(footprint "LibraryCANLED:K104K10X7RF5UH5_VIS"
 		(layer "F.Cu")
 		(at 177.5 68.499995 90)
@@
 		(embedded_fonts no)
 	)
-	(footprint "Package_DIP:DIP-18_W7.62mm_LongPads"
+	(footprint "LibraryCANLED:DIP-18_W7.62mm_LongPads"
 		(layer "F.Cu")
 		(at 143.81 97.58 180)
@@
 		)
 	)
-	(footprint "2604-1103-1:CONN3_2604-1103_WAG"
+	(footprint "LibraryCANLED:CONN3_2604-1103_WAG"
 		(layer "F.Cu")
 		(at 189.5 57.199999 180)
@@
 		(embedded_fonts no)
 	)
-	(footprint "2604-1103-1:CONN3_2604-1103_WAG"
+	(footprint "LibraryCANLED:CONN3_2604-1103_WAG"
 		(layer "F.Cu")
 		(at 169.9451 57.2 180)
@@
 		(embedded_fonts no)
 	)
-	(footprint "Capacitor_THT:C_Disc_D6.0mm_W2.5mm_P5.00mm"
+	(footprint "LibraryCANLED:C_Disc_D6.0mm_W2.5mm_P5.00mm"
 		(layer "F.Cu")
 		(at 158 88.5 180)
@@
 		)
 	)
-	(footprint "LED_THT:LED_D4.0mm"
+	(footprint "LibraryCANLED:LED_D4.0mm"
 		(layer "F.Cu")
 		(at 173.23 77)
@@
 		)
 	)
-	(footprint "Connector_PinHeader_2.54mm:PinHeader_1x02_P2.54mm_Vertical"
+	(footprint "LibraryCANLED:PinHeader_1x02_P2.54mm_Vertical"
 		(layer "F.Cu")
 		(at 159.5 63.725)
@@
 		)
 	)
-	(footprint "LED_THT:LED_D4.0mm"
+	(footprint "LibraryCANLED:LED_D4.0mm"
 		(layer "F.Cu")
 		(at 167.23 77)
@@
 		)
 	)
-	(footprint "Capacitor_THT:C_Disc_D5.0mm_W2.5mm_P5.00mm"
+	(footprint "LibraryCANLED:C_Disc_D5.0mm_W2.5mm_P5.00mm"
 		(layer "F.Cu")
 		(at 131.5 83 90)
@@
 		)
 	)
-	(footprint "footprints:K104K10X7RF5UH5_VIS"
+	(footprint "LibraryCANLED:K104K10X7RF5UH5_VIS"
 		(layer "F.Cu")
 		(at 125 65.5 -90)
@@
 		(embedded_fonts no)
 	)
-	(footprint "Resistor_THT:R_Axial_DIN0207_L6.3mm_D2.5mm_P10.16mm_Horizontal"
+	(footprint "LibraryCANLED:R_Axial_DIN0207_L6.3mm_D2.5mm_P10.16mm_Horizontal"
 		(layer "F.Cu")
 		(at 160.58 97 180)
@@
 		)
 	)
-	(footprint "2604-1104-1:CONN4_2604-1104_WAG"
+	(footprint "LibraryCANLED:CONN4_2604-1104_WAG"
 		(layer "F.Cu")
 		(at 130.9451 57.5 180)
@@
 		(embedded_fonts no)
 	)
-	(footprint "Diode_THT:D_DO-41_SOD81_P10.16mm_Horizontal"
+	(footprint "LibraryCANLED:D_DO-41_SOD81_P10.16mm_Horizontal"
 		(layer "F.Cu")
 		(at 180.92 79.5)
@@
 		)
 	)
-	(footprint "Capacitor_THT:C_Disc_D5.0mm_W2.5mm_P5.00mm"
+	(footprint "LibraryCANLED:C_Disc_D5.0mm_W2.5mm_P5.00mm"
 		(layer "F.Cu")
 		(at 131.5 91 90)
@@
 		)
 	)
-	(footprint "Capacitor_THT:C_Disc_D5.0mm_W2.5mm_P5.00mm"
+	(footprint "LibraryCANLED:C_Disc_D5.0mm_W2.5mm_P5.00mm"
 		(layer "F.Cu")
 		(at 154 82 90)
@@
 		)
 	)
-	(footprint "Connector_IDC:IDC-Header_2x03_P2.54mm_Vertical"
+	(footprint "LibraryCANLED:IDC-Header_2x03_P2.54mm_Vertical"
 		(layer "F.Cu")
 		(at 181.42 93.04 90)
@@
 		)
 	)
-	(footprint "Capacitor_THT:C_Disc_D5.0mm_W2.5mm_P5.00mm"
+	(footprint "LibraryCANLED:C_Disc_D5.0mm_W2.5mm_P5.00mm"
 		(layer "F.Cu")
 		(at 158.5 77 -90)
@@
 		)
 	)
-	(footprint "ABL-16.000MHZ-B2:XTAL_HC49P488W46L1150T500H350"
+	(footprint "LibraryCANLED:XTAL_HC49P488W46L1150T500H350"
 		(layer "F.Cu")
 		(at 126 86 -90)
@@
 		(embedded_fonts no)
 	)
-	(footprint "Jumper:SolderJumper-2_P1.3mm_Open_Pad1.0x1.5mm"
+	(footprint "LibraryCANLED:SolderJumper-2_P1.3mm_Open_Pad1.0x1.5mm"
 		(layer "F.Cu")
 		(at 126 95)
@@
 		(embedded_fonts no)
 	)
-	(footprint "2604-1103-1:CONN3_2604-1103_WAG"
+	(footprint "LibraryCANLED:CONN3_2604-1103_WAG"
 		(layer "F.Cu")
 		(at 150.5 57.199999 180)
@@
 		(embedded_fonts no)
 	)
-	(footprint "Package_DIP:DIP-28_W7.62mm"
+	(footprint "LibraryCANLED:DIP-28_W7.62mm"
 		(layer "F.Cu")
 		(at 113.38 64.34)
